File: pcb/pcb.kicad_sch (KiCad schematic)
At the start: 0 parts

Commit message: Added PCB Layout
Parts:
- added C1: 1uF, Capacitor_SMD:C_0805_2012Metric, symbol Device:C
- added C2, C3, C4: 0.1uF, Capacitor_SMD:C_0805_2012Metric, symbol Device:C
- added C5, C6: 10pF, Capacitor_SMD:C_0805_2012Metric, symbol Device:C_Small
- added D1, D10, D11, D12, D13, D14, D15, D16, D17, D18, D19, D2, D20, D21, D22, D23, D24, D25, D26, D27, D28, D29, D3, D30, D31, D32, D33, D34, D35, D36, D37, D38, D39, D4, D40, D41, D42, D43, D44, D45, D46, D47, D48, D49, D5, D50, D51, D52, D53, D54, D55, D56, D57, D58, D59, D6, D60, D61, D62, D63, D64, D65, D66, D67, D68, D7, D8, D9: 1N4148WT, Diode_SMD:D_SOD-123, symbol Diode:1N4148WT
- added F1: 500mA, Fuse:Fuse_1206_3216Metric, symbol Device:Polyfuse_Small
- added J1: USB_C_Receptacle_USB2.0_14P, Connector_USB:USB_C_Receptacle_HRO_TYPE-C-31-M-17, symbol Connector:USB_C_Receptacle_USB2.0_14P
- added R1, R2: 22, Resistor_SMD:R_0805_2012Metric, symbol Device:R_Small
- added R3, R4: 10k, Resistor_SMD:R_0805_2012Metric, symbol Device:R_Small
- added R5, R6: 5.1k, Resistor_SMD:R_0805_2012Metric, symbol Device:R_Small
- added SW0: SW_Push, Button_Switch_SMD:SW_SPST_B3S-1000, symbol Switch:SW_Push
- added SW1, SW10, SW11, SW12, SW13, SW14, SW17, SW18, SW19, SW2, SW20, SW21, SW22, SW23, SW24, SW25, SW26, SW27, SW28, SW29, SW3, SW32, SW33, SW34, SW35, SW36, SW37, SW38, SW39, SW4, SW40, SW41, SW42, SW43, SW46, SW47, SW48, SW49, SW5, SW50, SW51, SW52, SW53, SW54, SW55, SW57, SW58, SW6, SW66, SW67, SW68, SW7, SW8, SW9: SW_Push_45deg, Button_Switch_Keyboard:SW_Cherry_MX_1.00u_PCB, symbol Switch:SW_Push_45deg
- added SW15: SW_Push_45deg, Button_Switch_Keyboard:SW_Cherry_MX_2.00u_PCB, symbol Switch:SW_Push_45deg
- added SW16, SW30: SW_Push_45deg, Button_Switch_Keyboard:SW_Cherry_MX_1.50u_PCB, symbol Switch:SW_Push_45deg
- added SW31, SW56: SW_Push_45deg, Button_Switch_Keyboard:SW_Cherry_MX_1.75u_PCB, symbol Switch:SW_Push_45deg
- added SW44, SW45: SW_Push_45deg, Button_Switch_Keyboard:SW_Cherry_MX_2.25u_PCB, symbol Switch:SW_Push_45deg
- added SW59, SW60, SW61: SW_Push_45deg, Button_Switch_Keyboard:SW_Cherry_MX_1.25u_PCB, symbol Switch:SW_Push_45deg
- added SW62: SW_Push_45deg, Button_Switch_Keyboard:SW_Cherry_MX_6.25u_PCB, symbol Switch:SW_Push_45deg
- added SW63, SW64, SW65: SW_Push_45deg, Button_Switch_Keyboard:SW_Cherry_MX_1.00u_Plate, symbol Switch:SW_Push_45deg
- added U1: ATmega32U4-A, Package_QFP:TQFP-44_10x10mm_P0.8mm, symbol MCU_Microchip_ATmega:ATmega32U4-A
- added Y1: 16MHz, Crystal:Crystal_SMD_3225-4Pin_3.2x2.5mm, symbol Device:Crystal_GND24_Small
Connections:
- new net: D53.2 (A), SW53.1
- new net: D23.2 (A), SW23.1
- new net: D66.2 (A), SW66.1
- new net: D65.2 (A), SW65.1
- new net: D55.2 (A), SW55.1
- new net: D5.2 (A), SW5.1
- new net: D38.2 (A), SW38.1
- new net: D26.2 (A), SW26.1
- new net: D42.2 (A), SW42.1
- new net: D24.2 (A), SW24.1
- new net: D6.2 (A), SW6.1
- new net: D9.2 (A), SW9.1
- new net: D29.2 (A), SW29.1
- new net: R4.2, U1.33 (~{HWB}/PE2)
- new net: D34.2 (A), SW34.1
- new net: D30.2 (A), SW30.1
- new net: D39.2 (A), SW39.1
- new net: D33.2 (A), SW33.1
- new net: R2.2, U1.3 (D-)
- new net: C1.1, U1.6 (UCAP)
- new net: D12.2 (A), SW12.1
- new net: D28.2 (A), SW28.1
- new net: D57.2 (A), SW57.1
- new net: D13.2 (A), SW13.1
- new net: D1.2 (A), SW1.1
- new net: D64.2 (A), SW64.1
- new net: D62.2 (A), SW62.1
- new net: D59.2 (A), SW59.1
- new net: D15.2 (A), SW15.1
- new net: D31.2 (A), SW31.1
- new net: D67.2 (A), SW67.1
- new net: D32.2 (A), SW32.1
- new net: D61.2 (A), SW61.1
- new net: D19.2 (A), SW19.1
- new net: D18.2 (A), SW18.1
- new net: D36.2 (A), SW36.1
- new net: D11.2 (A), SW11.1
- new net: C6.2, U1.17 (XTAL1), Y1.1
- new net: C5.2, U1.16 (XTAL2), Y1.3
- new net: D45.2 (A), SW45.1
- new net: D50.2 (A), SW50.1
- new net: D17.2 (A), SW17.1
- new net: D52.2 (A), SW52.1
- new net: D58.2 (A), SW58.1
- new net: D44.2 (A), SW44.1
- new net: D41.2 (A), SW41.1
- new net: D46.2 (A), SW46.1
- new net: D14.2 (A), SW14.1
- new net: D37.2 (A), SW37.1
- new net: D43.2 (A), SW43.1
- new net: D21.2 (A), SW21.1
- new net: D54.2 (A), SW54.1
- new net: D49.2 (A), SW49.1
- new net: D8.2 (A), SW8.1
- new net: D68.2 (A), SW68.1
- new net: D20.2 (A), SW20.1
- new net: D2.2 (A), SW2.1
- new net: D4.2 (A), SW4.1
- new net: R3.1, SW0.2, U1.13 (~{RESET})
- new net: R1.2, U1.4 (D+)
- new net: D63.2 (A), SW63.1
- new net: J1.B5 (CC2), R6.2
- new net: D51.2 (A), SW51.1
- new net: D16.2 (A), SW16.1
- new net: D7.2 (A), SW7.1
- new net: D48.2 (A), SW48.1
- new net: D60.2 (A), SW60.1
- new net: D3.2 (A), SW3.1
- new net: D35.2 (A), SW35.1
- new net: D27.2 (A), SW27.1
- new net: D40.2 (A), SW40.1
- new net: F1.1, J1.A4 (VBUS), J1.A9 (VBUS), J1.B4 (VBUS), J1.B9 (VBUS)
- new net: J1.A5 (CC1), R5.2
- new net: D56.2 (A), SW56.1
- new net: D22.2 (A), SW22.1
- new net: D10.2 (A), SW10.1
- new net: D47.2 (A), SW47.1
- new net: D25.2 (A), SW25.1
- new net +5V: C2.1, C3.1, C4.1, F1.2, R3.2, U1.14 (VCC), U1.2 (UVCC), U1.24 (AVCC), U1.34 (VCC), U1.44 (AVCC), U1.7 (VBUS)
- new net COLUMN1: SW1.2, SW16.2, SW31.2, SW45.2, SW59.2, U1.29 (PB5)
- new net COLUMN10: SW10.2, SW25.2, SW40.2, SW54.2, SW68.2, U1.25 (PD4)
- new net COLUMN11: SW11.2, SW26.2, SW41.2, SW55.2, U1.22 (PD5)
- new net COLUMN12: SW12.2, SW27.2, SW42.2, SW56.2, U1.26 (PD6)
- new net COLUMN13: SW13.2, SW28.2, SW43.2, SW57.2, U1.27 (PD7)
- new net COLUMN14: SW14.2, SW29.2, SW44.2, SW58.2, U1.41 (PF0)
- new net COLUMN15: SW15.2, SW30.2, U1.40 (PF1)
- new net COLUMN2: SW17.2, SW2.2, SW32.2, SW46.2, SW60.2, U1.30 (PB6)
- new net COLUMN3: SW18.2, SW3.2, SW33.2, SW47.2, SW61.2, U1.12 (PB7)
- new net COLUMN4: SW19.2, SW34.2, SW4.2, SW48.2, SW62.2, U1.31 (PC6)
- new net COLUMN5: SW20.2, SW35.2, SW49.2, SW5.2, SW63.2, U1.32 (PC7)
- new net COLUMN6: SW21.2, SW36.2, SW50.2, SW6.2, SW64.2, U1.18 (PD0)
- new net COLUMN7: SW22.2, SW37.2, SW51.2, SW65.2, SW7.2, U1.19 (PD1)
- new net COLUMN8: SW23.2, SW38.2, SW52.2, SW66.2, SW8.2, U1.20 (PD2)
- new net COLUMN9: SW24.2, SW39.2, SW53.2, SW67.2, SW9.2, U1.21 (PD3)
- new net D+: J1.A6 (D+), J1.B6 (D+), R1.1
- new net D-: J1.A7 (D-), J1.B7 (D-), R2.1
- new net GND: C1.2, C2.2, C3.2, C4.2, C5.1, C6.1, J1.A1 (GND), J1.A12 (GND), J1.B1 (GND), J1.B12 (GND), J1.S1 (SHIELD), R4.1, R5.1, R6.1, SW0.1, U1.15 (GND), U1.23 (GND), U1.35 (GND), U1.43 (GND), U1.5 (UGND), Y1.2, Y1.4
- new net ROW1: D1.1 (K), D10.1 (K), D11.1 (K), D12.1 (K), D13.1 (K), D14.1 (K), D15.1 (K), D2.1 (K), D3.1 (K), D4.1 (K), D5.1 (K), D6.1 (K), D7.1 (K), D8.1 (K), D9.1 (K), U1.8 (PB0)
- new net ROW2: D16.1 (K), D17.1 (K), D18.1 (K), D19.1 (K), D20.1 (K), D21.1 (K), D22.1 (K), D23.1 (K), D24.1 (K), D25.1 (K), D26.1 (K), D27.1 (K), D28.1 (K), D29.1 (K), D30.1 (K), U1.9 (PB1)
- new net ROW3: D31.1 (K), D32.1 (K), D33.1 (K), D34.1 (K), D35.1 (K), D36.1 (K), D37.1 (K), D38.1 (K), D39.1 (K), D40.1 (K), D41.1 (K), D42.1 (K), D43.1 (K), D44.1 (K), U1.10 (PB2)
- new net ROW4: D45.1 (K), D46.1 (K), D47.1 (K), D48.1 (K), D49.1 (K), D50.1 (K), D51.1 (K), D52.1 (K), D53.1 (K), D54.1 (K), D55.1 (K), D56.1 (K), D57.1 (K), D58.1 (K), U1.11 (PB3)
- new net ROW5: D59.1 (K), D60.1 (K), D61.1 (K), D62.1 (K), D63.1 (K), D64.1 (K), D65.1 (K), D66.1 (K), D67.1 (K), D68.1 (K), U1.28 (PB4)
